File: schematic.brd (EAGLE design)
At the start: 160 x 100 mm, 56 parts, among them J1 FTDI_DEVICERA_SMT, M1 WIRELESS-NRF24L01, Q1 8MHz, T1 NMOS, T2 NMOS, T3 NMOS, T4 NMOS, U1 ATMEGA328P_TQFP, U2 GY-521MPU6050, U3 TPS63060

Commit message: Changed voltage divider values
Parts:
- R2: value 150K -> 50K
- R3: value 50K -> 150K
- S2: value PUSH_BUTT -> (none); device quad:TACTILE-SWITCH-SMD -> adafruit:PUSHBUTTON_SMD_SJ
- moved S2 256.8 mm to (-74.1, -190.6)
Connections:
- net GND: now also S2.P$1; no longer S2.1
- net N$2: now also S2.P$2; no longer S2.3
Changed lines of the file:
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@@
 <element name="LED4" library="led" library_urn="urn:adsk.eagle:library:259" package="SMARTLED-TTW" package3d_urn="urn:adsk.eagle:package:15825/1" value="YELLOW" x="-20.32" y="62.23"/>
 <element name="M1" library="quad" package="WIRELESS-NRF24L01" value="WIRELESS-NRF24L01" x="-44.45" y="10.16"/>
-<element name="R2" library="resistor" library_urn="urn:adsk.eagle:library:348" package="M2309" package3d_urn="urn:adsk.eagle:package:26085/1" value="150K" x="-27.94" y="48.26"/>
+<element name="R2" library="resistor" library_urn="urn:adsk.eagle:library:348" package="M2309" package3d_urn="urn:adsk.eagle:package:26085/1" value="50K" x="-27.94" y="48.26"/>
 <element name="S1" library="SparkFun" package="SWITCH-SPST-SMD-A" value="MAIN_SWITCH" x="-27.94" y="62.23"/>
-<element name="S2" library="quad" package="TACTILE-SWITCH-SMD" value="PUSH_BUTT" x="-36.83" y="63.5">
-<attribute name="PROD_ID" value="SWCH-08247" x="-36.83" y="63.5" size="1.778" layer="27" display="off"/>
-</element>
 <element name="U$1" library="quad" package="JST_CONNECTOR_FEMALE" value="JST_CONNECTOR_FEMALE" x="-34.29" y="55.88"/>
 <element name="U$10" library="quad" package="JST_CONNECTOR_FEMALE" value="JST_CONNECTOR_FEMALE" x="-49.53" y="55.88"/>
@@
 </element>
 <element name="C17" library="resistor" library_urn="urn:adsk.eagle:library:348" package="C0201" package3d_urn="urn:adsk.eagle:package:26209/1" value="0.1uF" x="-79.297834375" y="-118.6854625"/>
-<element name="R3" library="resistor" library_urn="urn:adsk.eagle:library:348" package="R0805" package3d_urn="urn:adsk.eagle:package:26059/1" value="50K" x="-78.4424375" y="-130.3440625"/>
+<element name="R3" library="resistor" library_urn="urn:adsk.eagle:library:348" package="R0805" package3d_urn="urn:adsk.eagle:package:26059/1" value="150K" x="-78.4424375" y="-130.3440625"/>
 <element name="C4" library="rcl" library_urn="urn:adsk.eagle:library:334" package="C0603" package3d_urn="urn:adsk.eagle:package:23616/2" value="0.1uF" x="-77.757503125" y="-135.8558625">
 <attribute name="SPICEPREFIX" value="C" x="-77.757503125" y="-135.8558625" size="1.778" layer="27" display="off"/>
@@
 </element>
 <element name="C16" library="resistor" library_urn="urn:adsk.eagle:library:348" package="C0805K" package3d_urn="urn:adsk.eagle:package:26201/1" value="10uF" x="-78.689225" y="-184.82673125"/>
+<element name="S2" library="adafruit" package="PUSHBUTTON_SMD_SJ" value="" x="-74.107496875" y="-190.594996875"/>
 </elements>
 <signals>
@@
 <signal name="N$2">
 <contactref element="U1" pad="29"/>
-<contactref element="S2" pad="3"/>
 <contactref element="R7" pad="1"/>
 <contactref element="C9" pad="2"/>
+<contactref element="S2" pad="P$2"/>
+<wire x1="-77.107496875" y1="-190.594996875" x2="-76.907503125" y2="-140.7326625" width="0" layer="19" extent="1-1"/>
 <wire x1="-71.884909375" y1="-86.721721875" x2="-76.907503125" y2="-140.7326625" width="0" layer="19" extent="1-1"/>
 <wire x1="-38.5" y1="33.5026" x2="-71.884909375" y2="-86.721721875" width="0" layer="19" extent="1-1"/>
-<wire x1="-39.624" y1="61.595" x2="-38.5" y2="33.5026" width="0" layer="19" extent="1-1"/>
 </signal>
 <signal name="GND">
-<contactref element="S2" pad="1"/>
 <contactref element="U1" pad="3"/>
 <contactref element="U1" pad="5"/>
@@
 <contactref element="C8" pad="2"/>
 <contactref element="C16" pad="2"/>
+<contactref element="S2" pad="P$1"/>
 <wire x1="-76.907503125" y1="-169.9934625" x2="-76.907503125" y2="-174.8702625" width="0" layer="19" extent="1-1"/>
 <wire x1="-76.907503125" y1="-179.7470625" x2="-76.907503125" y2="-174.8702625" width="0" layer="19" extent="1-1"/>
 <wire x1="-77.689225" y1="-184.82673125" x2="-76.907503125" y2="-179.7470625" width="0" layer="19" extent="1-1"/>
+<wire x1="-71.107496875" y1="-190.594996875" x2="-77.689225" y2="-184.82673125" width="0" layer="19" extent="1-1"/>
 <wire x1="-76.907503125" y1="-160.2398625" x2="-76.907503125" y2="-169.9934625" width="0" layer="19" extent="1-1"/>
 <wire x1="-76.907503125" y1="-155.3630625" x2="-76.907503125" y2="-160.2398625" width="0" layer="19" extent="1-1"/>
@@
 <wire x1="-17.78" y1="35.48" x2="-20.32" y2="35.48" width="0" layer="19" extent="1-1"/>
 <wire x1="-34.29" y1="54.88" x2="-20.32" y2="35.48" width="0" layer="19" extent="1-1"/>
-<wire x1="-39.624" y1="65.405" x2="-34.29" y2="54.88" width="0" layer="19" extent="1-1"/>
-<wire x1="-37.15" y1="67.58" x2="-39.624" y2="65.405" width="0" layer="19" extent="1-1"/>
+<wire x1="-37.15" y1="67.58" x2="-34.29" y2="54.88" width="0" layer="19" extent="1-1"/>
 <wire x1="-30.9" y1="72.39" x2="-37.15" y2="67.58" width="0" layer="19" extent="1-1"/>
 <wire x1="-26.825" y1="69.18" x2="-30.9" y2="72.39" width="0" layer="19" extent="1-1"/>
@@
 <wire x1="-20.32" y1="62.73" x2="-24.9" y2="67.105" width="0" layer="19" extent="1-1"/>
 <wire x1="-15.24" y1="62.73" x2="-20.32" y2="62.73" width="0" layer="19" extent="1-1"/>
-<wire x1="-43.6" y1="72.39" x2="-39.624" y2="65.405" width="0" layer="19" extent="1-1"/>
+<wire x1="-43.6" y1="72.39" x2="-37.15" y2="67.58" width="0" layer="19" extent="1-1"/>
 <wire x1="-49.85" y1="67.58" x2="-43.6" y2="72.39" width="0" layer="19" extent="1-1"/>
 <wire x1="-57.42" y1="62.23" x2="-49.85" y2="67.58" width="0" layer="19" extent="1-1"/>

Commit message: added slide switch
Parts:
- S1: value MAIN_SWITCH -> SLIDING_SIWTCH; device SparkFun:SWITCH-SPST-SMD-A -> wurth:SLIDE_SWITCH
- moved S1 256.5 mm to (-83.6, -188.2)
Connections:
- net N$8: now also S1.P$5; no longer S1.2
- net VCC: now also S1.P$6; no longer S1.1
Changed lines of the file:
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@@
 <layer number="59" name="tCarbon" color="7" fill="1" visible="no" active="no"/>
 <layer number="60" name="bCarbon" color="7" fill="1" visible="no" active="no"/>
+<layer number="88" name="SimResults" color="9" fill="1" visible="no" active="no"/>
+<layer number="89" name="SimProbes" color="9" fill="1" visible="no" active="no"/>
 <layer number="90" name="Modules" color="5" fill="1" visible="no" active="no"/>
 <layer number="91" name="Nets" color="2" fill="1" visible="no" active="no"/>
@@
 <element name="M1" library="quad" package="WIRELESS-NRF24L01" value="WIRELESS-NRF24L01" x="-44.45" y="10.16"/>
 <element name="R2" library="resistor" library_urn="urn:adsk.eagle:library:348" package="M2309" package3d_urn="urn:adsk.eagle:package:26085/1" value="50K" x="-27.94" y="48.26"/>
-<element name="S1" library="SparkFun" package="SWITCH-SPST-SMD-A" value="MAIN_SWITCH" x="-27.94" y="62.23"/>
 <element name="U$1" library="quad" package="JST_CONNECTOR_FEMALE" value="JST_CONNECTOR_FEMALE" x="-34.29" y="55.88"/>
 <element name="U$10" library="quad" package="JST_CONNECTOR_FEMALE" value="JST_CONNECTOR_FEMALE" x="-49.53" y="55.88"/>
@@
 <element name="C16" library="resistor" library_urn="urn:adsk.eagle:library:348" package="C0805K" package3d_urn="urn:adsk.eagle:package:26201/1" value="10uF" x="-78.689225" y="-184.82673125"/>
 <element name="S2" library="adafruit" package="PUSHBUTTON_SMD_SJ" value="" x="-74.107496875" y="-190.594996875"/>
+<element name="S1" library="wurth" package="SLIDE_SWITCH" value="SLIDING_SIWTCH" x="-83.642453125" y="-188.196575"/>
 </elements>
 <signals>
@@
 <contactref element="U$13" pad="+"/>
 <contactref element="D4" pad="NEG"/>
-<contactref element="S1" pad="1"/>
 <contactref element="R1" pad="1"/>
 <contactref element="C1" pad="1"/>
+<contactref element="S1" pad="P$6"/>
+<wire x1="-81.142453125" y1="-191.196575" x2="-79.342440625" y2="-111.721646875" width="0" layer="19" extent="1-1"/>
 <wire x1="-71.884909375" y1="-29.01904375" x2="-79.342440625" y2="-111.721646875" width="0" layer="19" extent="1-1"/>
 <wire x1="-54.61" y1="56.88" x2="-71.884909375" y2="-29.01904375" width="0" layer="19" extent="1-1"/>
@@
 <wire x1="-67.31" y1="63.78" x2="-64.5" y2="62.23" width="0" layer="19" extent="1-1"/>
 <wire x1="-69.85" y1="63.78" x2="-67.31" y2="63.78" width="0" layer="19" extent="1-1"/>
-<wire x1="-30.19" y1="60.48" x2="-39.37" y2="56.88" width="0" layer="19" extent="1-1"/>
-<wire x1="-25.9" y1="67.105" x2="-30.19" y2="60.48" width="0" layer="19" extent="1-1"/>
+<wire x1="-25.09" y1="48.26" x2="-39.37" y2="56.88" width="0" layer="19" extent="1-1"/>
+<wire x1="-25.9" y1="67.105" x2="-39.37" y2="56.88" width="0" layer="19" extent="1-1"/>
 <wire x1="-25.4" y1="67.105" x2="-25.9" y2="67.105" width="0" layer="19" extent="1-1"/>
 <wire x1="-16.51" y1="70.13" x2="-25.4" y2="67.105" width="0" layer="19" extent="1-1"/>
 <wire x1="-13.97" y1="70.13" x2="-16.51" y2="70.13" width="0" layer="19" extent="1-1"/>
-<wire x1="-25.09" y1="48.26" x2="-30.19" y2="60.48" width="0" layer="19" extent="1-1"/>
 </signal>
 <signal name="N$2">
@@
 <wire x1="-25.08" y1="72.66" x2="-37.7" y2="24.9174" width="0" layer="19" extent="1-1"/>
 </signal>
-<signal name="N$8">
-<contactref element="S1" pad="2"/>
-<contactref element="U$1" pad="+"/>
-<wire x1="-34.29" y1="56.88" x2="-28.69" y2="60.48" width="0" layer="19" extent="1-1"/>
-</signal>
 <signal name="N$10">
 <contactref element="R1" pad="2"/>
@@
 <wire x1="-45.3" y1="72.39" x2="-42.3926" y2="27.21" width="0" layer="19" extent="1-1"/>
 </signal>
+<signal name="N$8">
+<contactref element="U$1" pad="+"/>
+<contactref element="S1" pad="P$5"/>
+<wire x1="-83.642453125" y1="-191.196575" x2="-34.29" y2="56.88" width="0" layer="19" extent="1-1"/>
+</signal>
 </signals>
