File: schematic.brd (EAGLE design)
At the start: 160 x 100 mm, 56 parts, among them J1 FTDI_DEVICERA_SMT, M1 WIRELESS-NRF24L01, Q1 8MHz, T1 NMOS, T2 NMOS, T3 NMOS, T4 NMOS, U1 ATMEGA328P_TQFP, U2 GY-521MPU6050, U3 LTC3534

Commit message: Fixed LED package
Parts:
- LED3, LED4: device led:SMARTLED-TTW -> led:SML0603
- moved LED3 267.4 mm to (-255.3, -55.5)
- moved LED4 264.6 mm to (-255.3, -59.4)
- moved LED2 196.2 mm to (-255.3, -51.7)
- moved LED1 127.7 mm to (-255.3, -47.9)
Connections:
- net GND: now also LED3.C, LED4.C; no longer LED3.C@1, LED4.C@1
- net N$12: now also LED3.A; no longer LED3.A@1
- net N$13: now also LED4.A; no longer LED4.A@1
Changed lines of the file:
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@@
 <attribute name="PROD_ID" value="CONN-08971" x="-24.13" y="30.48" size="1.778" layer="27" display="off"/>
 </element>
-<element name="LED3" library="led" library_urn="urn:adsk.eagle:library:259" package="SMARTLED-TTW" package3d_urn="urn:adsk.eagle:package:15825/1" value="YELLOW" x="-15.24" y="62.23"/>
-<element name="LED4" library="led" library_urn="urn:adsk.eagle:library:259" package="SMARTLED-TTW" package3d_urn="urn:adsk.eagle:package:15825/1" value="YELLOW" x="-20.32" y="62.23"/>
 <element name="M1" library="quad" package="WIRELESS-NRF24L01" value="WIRELESS-NRF24L01" x="-44.45" y="10.16"/>
 <element name="U$1" library="quad" package="JST_CONNECTOR_FEMALE" value="JST_CONNECTOR_FEMALE" x="-34.29" y="55.88"/>
@@
 <attribute name="SPICEPREFIX" value="R" x="-133.350659375" y="22.44051875" size="0.1" layer="27" display="off"/>
 </element>
-<element name="LED1" library="led" library_urn="urn:adsk.eagle:library:259" package="SML0603" package3d_urn="urn:adsk.eagle:package:15832/1" value="RED" x="-132.76575" y="-12.06208125"/>
-<element name="LED2" library="led" library_urn="urn:adsk.eagle:library:259" package="SML0603" package3d_urn="urn:adsk.eagle:package:15832/1" value="RED" x="-174.76658125" y="127.168528125"/>
 <element name="R10" library="resistor" library_urn="urn:adsk.eagle:library:348" package="R0603" package3d_urn="urn:adsk.eagle:package:26057/1" value="10K" x="-175.351490625" y="122.19670625"/>
 <element name="R13" library="resistor" library_urn="urn:adsk.eagle:library:348" package="R0603" package3d_urn="urn:adsk.eagle:package:26057/1" value="10K" x="-175.351490625" y="117.31990625"/>
@@
 <attribute name="SPICEPREFIX" value="C" x="-254.903171875" y="-38.13764375" size="1.778" layer="27" display="off"/>
 </element>
+<element name="LED1" library="led" library_urn="urn:adsk.eagle:library:259" package="SML0603" package3d_urn="urn:adsk.eagle:package:15832/1" value="RED" x="-255.318259375" y="-47.859265625"/>
+<element name="LED2" library="led" library_urn="urn:adsk.eagle:library:259" package="SML0603" package3d_urn="urn:adsk.eagle:package:15832/1" value="RED" x="-255.318259375" y="-51.7040875"/>
+<element name="LED3" library="led" library_urn="urn:adsk.eagle:library:259" package="SML0603" package3d_urn="urn:adsk.eagle:package:15832/1" value="YELLOW" x="-255.318259375" y="-55.5489125"/>
+<element name="LED4" library="led" library_urn="urn:adsk.eagle:library:259" package="SML0603" package3d_urn="urn:adsk.eagle:package:15832/1" value="YELLOW" x="-255.318259375" y="-59.393734375"/>
 </elements>
 <signals>
@@
 <contactref element="T3" pad="2"/>
 <contactref element="T4" pad="2"/>
-<contactref element="LED3" pad="C@1"/>
-<contactref element="LED4" pad="C@1"/>
 <contactref element="C12" pad="2"/>
 <contactref element="C13" pad="2"/>
-<contactref element="LED1" pad="C"/>
-<contactref element="LED2" pad="C"/>
 <contactref element="R13" pad="1"/>
 <contactref element="R14" pad="1"/>
@@
 <contactref element="R15" pad="1"/>
 <contactref element="R16" pad="1"/>
+<contactref element="LED1" pad="C"/>
+<contactref element="LED2" pad="C"/>
+<contactref element="LED3" pad="C"/>
+<contactref element="LED4" pad="C"/>
 <wire x1="-256.753175" y1="31.291603125" x2="-256.753175" y2="6.907603125" width="0" layer="19" extent="1-1"/>
 <wire x1="-253.8682625" y1="41.045203125" x2="-256.753175" y2="31.291603125" width="0" layer="19" extent="1-1"/>
@@
 <wire x1="-256.753171875" y1="-27.74904375" x2="-253.8682625" y2="-22.87224375" width="0" layer="19" extent="1-1"/>
 <wire x1="-256.753171875" y1="-32.62584375" x2="-256.753171875" y2="-27.74904375" width="0" layer="19" extent="1-1"/>
+<wire x1="-256.068259375" y1="-47.859265625" x2="-256.753171875" y2="-32.62584375" width="0" layer="19" extent="1-1"/>
+<wire x1="-256.068259375" y1="-51.7040875" x2="-256.068259375" y2="-47.859265625" width="0" layer="19" extent="1-1"/>
+<wire x1="-256.068259375" y1="-55.5489125" x2="-256.068259375" y2="-51.7040875" width="0" layer="19" extent="1-1"/>
+<wire x1="-256.068259375" y1="-59.393734375" x2="-256.068259375" y2="-55.5489125" width="0" layer="19" extent="1-1"/>
 <wire x1="-203.748209375" y1="8.034984375" x2="-256.753175" y2="6.907603125" width="0" layer="19" extent="1-1"/>
 <wire x1="-199.303209375" y1="8.034984375" x2="-203.748209375" y2="8.034984375" width="0" layer="19" extent="1-1"/>
@@
 <wire x1="-176.201490625" y1="112.44310625" x2="-180.859021875" y2="97.19678125" width="0" layer="19" extent="1-1"/>
 <wire x1="-176.201490625" y1="117.31990625" x2="-176.201490625" y2="112.44310625" width="0" layer="19" extent="1-1"/>
-<wire x1="-175.51658125" y1="127.168528125" x2="-176.201490625" y2="117.31990625" width="0" layer="19" extent="1-1"/>
-<wire x1="-133.51575" y1="-12.06208125" x2="-175.424078125" y2="18.32343125" width="0" layer="19" extent="1-1"/>
-<wire x1="-57.15" y1="16.51" x2="-133.51575" y2="-12.06208125" width="0" layer="19" extent="1-1"/>
+<wire x1="-57.15" y1="16.51" x2="-175.424078125" y2="18.32343125" width="0" layer="19" extent="1-1"/>
 <wire x1="-42.3926" y1="28.81" x2="-57.15" y2="16.51" width="0" layer="19" extent="1-1"/>
 <wire x1="-42.3926" y1="30.41" x2="-42.3926" y2="28.81" width="0" layer="19" extent="1-1"/>
@@
 <wire x1="-43.6" y1="72.39" x2="-37.15" y2="67.58" width="0" layer="19" extent="1-1"/>
 <wire x1="-49.85" y1="67.58" x2="-43.6" y2="72.39" width="0" layer="19" extent="1-1"/>
-<wire x1="-20.32" y1="62.73" x2="-23.18" y2="72.66" width="0" layer="19" extent="1-1"/>
-<wire x1="-15.24" y1="62.73" x2="-20.32" y2="62.73" width="0" layer="19" extent="1-1"/>
 <wire x1="-62.55" y1="67.58" x2="-49.85" y2="67.58" width="0" layer="19" extent="1-1"/>
 </signal>
@@
 <contactref element="R1" pad="2"/>
 <contactref element="LED1" pad="A"/>
-<wire x1="-132.500659375" y1="35.33195625" x2="-132.01575" y2="-12.06208125" width="0" layer="19" extent="1-1"/>
+<wire x1="-254.568259375" y1="-47.859265625" x2="-132.500659375" y2="35.33195625" width="0" layer="19" extent="1-1"/>
 </signal>
 <signal name="N$11">
 <contactref element="R9" pad="1"/>
 <contactref element="LED2" pad="A"/>
-<wire x1="-174.01658125" y1="127.168528125" x2="-134.200659375" y2="31.034809375" width="0" layer="19" extent="1-1"/>
+<wire x1="-254.568259375" y1="-51.7040875" x2="-134.200659375" y2="31.034809375" width="0" layer="19" extent="1-1"/>
 </signal>
 <signal name="DEBUG_LED1">
@@
 </signal>
 <signal name="N$12">
-<contactref element="LED3" pad="A@1"/>
 <contactref element="R12" pad="1"/>
-<wire x1="-15.24" y1="61.73" x2="-134.200659375" y2="26.7376625" width="0" layer="19" extent="1-1"/>
+<contactref element="LED3" pad="A"/>
+<wire x1="-254.568259375" y1="-55.5489125" x2="-134.200659375" y2="26.7376625" width="0" layer="19" extent="1-1"/>
 </signal>
 <signal name="N$13">
-<contactref element="LED4" pad="A@1"/>
 <contactref element="R11" pad="1"/>
-<wire x1="-20.32" y1="61.73" x2="-134.200659375" y2="22.44051875" width="0" layer="19" extent="1-1"/>
+<contactref element="LED4" pad="A"/>
+<wire x1="-254.568259375" y1="-59.393734375" x2="-134.200659375" y2="22.44051875" width="0" layer="19" extent="1-1"/>
 </signal>
 <signal name="N$1">
