File: schematic.brd (EAGLE design)
At the start: 47 x 28 mm, 56 parts, among them J1 FTDI_DEVICERA_SMT, M1 WIRELESS-NRF24L01, Q1 8MHz, T1 NMOS, T2 NMOS, T3 NMOS, T4 NMOS, U1 ATMEGA328P_TQFP, U2 GY-521MPU6050, U3 LTC3534

Commit message: Started PCB design
Current plan: motor driver on bottom, RF module on bottom, need to space out top to make room for reset push button and debug LED
Parts:
- moved R4 273.2 mm to (11.8, 15.6)
- moved R5 272.8 mm to (13.2, 5.92)
- moved C2 272.5 mm to (11.8, 17.2)
- moved C5 270.9 mm to (14.2, 8.03), turned to 180 degrees
- moved C3 270.6 mm to (13.4, 19.1), turned to 180 degrees
- moved R6 269.9 mm to (12.1, 3.63)
- moved R8 268.1 mm to (11.1, 8.00), turned to 180 degrees
- moved C4 267.7 mm to (9.16, 5.78), turned to 180 degrees
- moved R7 265.3 mm to (8.41, 3.62)
- moved C6 260.7 mm to (5.37, 4.02)
- moved C7 260.2 mm to (5.27, 5.54)
- moved R10 219.7 mm to (15.4, 13.1), turned to 180 degrees
- moved C8 205.6 mm to (15.2, 10.3), turned to 90 degrees
- moved L1 198.3 mm to (6.39, 18.6), turned to 180 degrees
- moved S2 170.3 mm to (-8.80, 3.11)
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Routing:
- net GND: track 0.00 -> 122.4 mm, vias 0 -> 3
- net V_REG_OUT: track 0.00 -> 79.5 mm
- net PWR: track 0.00 -> 40.8 mm
- net TXD: track 0.00 -> 23.2 mm, vias 0 -> 2
- net RXD: track 0.00 -> 22.5 mm, vias 0 -> 2
- net SCL: track 0.00 -> 17.9 mm, vias 0 -> 2
- net SDA: track 0.00 -> 16.5 mm
- net N$18: track 0.00 -> 13.8 mm
- net N$16: track 0.00 -> 7.02 mm
- net N$19: track 0.00 -> 6.51 mm
- net N$8: track 0.00 -> 4.51 mm
- net N$9: track 0.00 -> 4.37 mm
- net N$20: track 0.00 -> 4.23 mm
- net N$14: track 0.00 -> 1.85 mm
