File: schematic - Copy.brd (EAGLE design)
At the start: 47 x 28 mm, 56 parts, among them J1 FTDI_DEVICERA_SMT, M1 WIRELESS-NRF24L01, Q1 8MHz, T1 NMOS, T2 NMOS, T3 NMOS, T4 NMOS, U1 ATMEGA328P_TQFP, U2 GY-521MPU6050, U3 LTC3534

Commit message: Restarting design
Parts:
- moved R3 268.3 mm to (12.0, 21.9), turned to 180 degrees
- moved R2 264.6 mm to (8.46, 21.8), turned to 180 degrees
- moved LED2 263.6 mm to (2.11, 4.90), turned to 270 degrees
- moved LED3 256.9 mm to (-20.3, 48.3)
- moved R15 256.6 mm to (-16.5, 64.8)
- moved R16 253.7 mm to (-21.6, 64.8)
- moved LED4 250.2 mm to (-29.2, 47.7), turned to 180 degrees
- moved LED1 239.9 mm to (-35.6, 48.3)
- moved C15 236.8 mm to (-29.2, 49.4)
- moved C14 225.4 mm to (-43.2, 59.7)
- moved C11 200.4 mm to (12.1, 4.24), turned to 90 degrees
- moved C9 198.4 mm to (9.53, 11.7), turned to 180 degrees
- moved C1 174.7 mm to (-16.5, 41.9)
- moved C10 158.0 mm to (-24.1, 54.6)
- moved R9 151.2 mm to (15.4, 4.06)
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Routing:
- net GND: track 153.6 -> 0.00 mm, vias 6 -> 0
- net V_REG_OUT: track 80.0 -> 0.00 mm, vias 1 -> 0
- net PWR: track 40.9 -> 0.00 mm
- net SCL: track 17.9 -> 0.00 mm, vias 2 -> 0
- net SDA: track 16.5 -> 0.00 mm
- net N$18: track 13.8 -> 0.00 mm
- net N$2: track 9.08 -> 0.00 mm
- net N$16: track 7.02 -> 0.00 mm
- net N$19: track 6.51 -> 0.00 mm
- net DTR: track 5.08 -> 0.00 mm, vias 1 -> 0
- net N$8: track 4.51 -> 0.00 mm
- net N$9: track 4.37 -> 0.00 mm
- net N$20: track 4.23 -> 0.00 mm
- net N$14: track 1.85 -> 0.00 mm
Other:
- outline, holes or cut-outs redrawn
