File: schematic-version5 - Jingbin.brd (EAGLE design)
At the start: 47 x 28 mm, 54 parts, among them J2 FTDI_DEVICE, M1 WIRELESS-NRF24L01, Q1 NX3225GD, T1 NMOS, T2 NMOS, T3 NMOS, T4 NMOS, U1 ATMEGA328P_TQFP, U2 GY-521MPU6050

Commit message: More adjustments to version4, version5 is empty
Parts:
- moved T1 103.4 mm to (-49.5, 59.7), turned to 0 degrees
- moved T2 102.8 mm to (-53.3, 59.7), flipped to the top, turned to 0 degrees
- moved T3 101.3 mm to (-57.1, 59.7), flipped to the top, turned to 0 degrees
- moved U$4 100.4 mm to (-58.4, 25.4), turned to 0 degrees
- moved T4 99.7 mm to (-61.0, 59.7), flipped to the top, turned to 0 degrees
- moved R10 99.6 mm to (-58.4, 49.5), turned to 0 degrees
- moved R11 98.4 mm to (-57.1, 54.6), turned to 0 degrees
- moved R12 98.0 mm to (-63.5, 49.5), turned to 0 degrees
- moved D1 92.2 mm to (-34.3, 59.7), flipped to the top, turned to 0 degrees
- moved D2 87.5 mm to (-36.8, 59.7), flipped to the top, turned to 0 degrees
- moved D3 84.6 mm to (-39.4, 59.7), flipped to the top, turned to 0 degrees
- moved R3 82.5 mm to (-41.9, 54.6), turned to 0 degrees
- moved D4 81.8 mm to (-41.9, 59.7), flipped to the top, turned to 0 degrees
- moved S2 80.9 mm to (-40.6, 25.4), turned to 0 degrees
- moved R1 80.4 mm to (-62.2, 54.6), turned to 0 degrees
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Routing:
- net GND: track 93.0 -> 0.00 mm, vias 18 -> 0
- net PWR: track 47.7 -> 0.00 mm, vias 1 -> 0
- net SDA: track 44.7 -> 0.00 mm, vias 3 -> 0
- net SCL: track 40.8 -> 0.00 mm, vias 3 -> 0
- net PWM1: track 25.5 -> 0.00 mm, vias 2 -> 0
- net V_REG_OUT: track 21.4 -> 0.00 mm
- net PWM2: track 20.4 -> 0.00 mm, vias 3 -> 0
- net TXD: track 18.0 -> 0.00 mm, vias 1 -> 0
- net RXD: track 16.6 -> 0.00 mm, vias 3 -> 0
- net N$2: track 15.9 -> 0.00 mm
- net PWM3: track 15.7 -> 0.00 mm, vias 3 -> 0
- net N$18: track 15.5 -> 0.00 mm, vias 2 -> 0
- net PWM4: track 11.2 -> 0.00 mm, vias 1 -> 0
- net DEBUG_LED2: track 10.7 -> 0.00 mm
- net N$3: track 8.79 -> 0.00 mm, vias 1 -> 0
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- removed copper zone on layer 16, net GND
- removed copper zone on layer 1, net PWR
- removed copper zone on layer 1, net V_REG_OUT
Other:
- outline, holes or cut-outs redrawn
- board text removed: "L1"
